Commit message: project finished

File: src/robot_2w_description/urdf/robot_2w_links/wheel.urdf.xacro (robot description, xacro)
@@ -31,5 +31,5 @@
         <parent link="${prefix}${parent}" />
         <child link="${prefix}${side}_wheel_link" />
-        <origin xyz="-0.02 ${flip*wheel_distance/2.0} -0.04" />
+        <origin xyz="0.0 ${flip*wheel_distance/2.0} -0.045" />
         <axis xyz="0 1 0" />
     </joint>
